File: class_e/class_e.kicad_pcb (KiCad board)
At the start: 4 copper layers, 64 x 46 mm, 52 parts, among them P201 CONN_01X04, P202 RCA_1, P301 CONN_01X03, P401 CONN_01X03, Q401 Q_NMOS_letters, Q402 Q_NMOS_letters, U201 STM32F334K, U301 LD1117S33TR, U401 UCC27524A, X201 CRYSTAL_SMD_4

Commit message: slight pcb changes, sent off to fab
Parts:
- moved C404 0.50 mm to (137.0, 72.0)
- moved C405 0.50 mm to (140.0, 72.0)
- moved C407 0.50 mm to (152.0, 72.0)
Routing:
- net GND: track 101.3 -> 99.0 mm, vias 98 -> 96
Other:
- board text added: "6+"
- board text removed: "12+"
